File: Open Op.sch (KiCad schematic (older format))
At the start: 6 parts, among them J3 Conn_01x04_Male, U1 Teensy3.6, U2 M25PX32-VMW, U3 TFT_TOUCH_SPI

Commit message: trying pins 0 and 1 for apa102
Changed lines of the file:
@@
 Text GLabel 3300 1050 0    50   Input ~ 0
 E4B
-Text GLabel 3300 4850 0    50   Input ~ 0
+Text GLabel 3300 950  0    50   Input ~ 0
 RGB_DATA
-Text GLabel 3300 4950 0    50   Input ~ 0
+Text GLabel 3300 850  0    50   Input ~ 0
 RGB_CLOCK
 Wire Wire Line
@@
 Wire Wire Line
 	5300 4050 6150 4050
-Text GLabel 3300 1250 0    50   Input ~ 0
+Text GLabel 3300 4950 0    50   Input ~ 0
 BATT_STAT2
-Text GLabel 3300 950  0    50   Input ~ 0
+Text GLabel 3300 4850 0    50   Input ~ 0
 BATT_STAT1
 Wire Wire Line
@@
 Wire Wire Line
 	2650 2150 3300 2150
-Text GLabel 3300 850  0    50   Input ~ 0
+Text GLabel 3300 1250 0    50   Input ~ 0
 REC_LED
 $Comp
@@
 SCL
 $Comp
-L power:+3V3 #PWR?
+L power:+3V3 #PWR0154
 U 1 1 5BA1378F
 P 6700 1700
-F 0 "#PWR?" H 6700 1550 50  0001 C CNN
+F 0 "#PWR0154" H 6700 1550 50  0001 C CNN
 F 1 "+3V3" H 6715 1873 50  0000 C CNN
 F 2 "" H 6700 1700 50  0001 C CNN
@@
 $EndComp
 $Comp
-L power:GND #PWR?
+L power:GND #PWR0155
 U 1 1 5BA13809
 P 6700 2000
-F 0 "#PWR?" H 6700 1750 50  0001 C CNN
+F 0 "#PWR0155" H 6700 1750 50  0001 C CNN
 F 1 "GND" H 6705 1827 50  0000 C CNN
 F 2 "" H 6700 2000 50  0001 C CNN
