File: SGTL5000.sch (KiCad schematic (older format))
At the start: 20 parts, among them J2 AudioJack3_Ground, U6 AP7313-1.8V, U7 SGTL5000

Commit message: mass rename
Parts:
- J2: footprint OpenOpParts:SJ1-3523N -> teensy_beats_parts:SJ1-3523N; symbol OpenOpParts:SJ1-3523N -> teensy_beats_parts:SJ1-3523N
- MK1: footprint OpenOpParts:AOM-6738P-R -> teensy_beats_parts:AOM-6738P-R
- RV1: footprint OpenOpParts:RV100F-30-4K1-B50K -> teensy_beats_parts:RV100F-30-4K1-B50K
- U6: symbol OpenOpParts:AP7313R-1.8V -> teensy_beats_parts:AP7313R-1.8V
Changed lines of the file:
@@
 	5450 4850 5450 4950
 $Comp
-L OpenOpParts:SJ1-3523N J?
+L teensy_beats_parts:SJ1-3523N J?
 U 1 1 5BAC3E4F
 P 7050 3850
@@
 F 0 "J2" H 6867 3779 50  0000 R CNN
 F 1 "AudioJack3_Ground" H 6867 3870 50  0000 R CNN
-F 2 "OpenOpParts:SJ1-3523N" H 7050 3850 50  0001 C CNN
+F 2 "teensy_beats_parts:SJ1-3523N" H 7050 3850 50  0001 C CNN
 F 3 "~" H 7050 3850 50  0001 C CNN
 	1    7050 3850
@@
 $EndComp
 $Comp
-L OpenOpParts:AP7313R-1.8V U?
+L teensy_beats_parts:AP7313R-1.8V U?
 U 1 1 5BAC54DA
 P 2250 2100
@@
 F 0 "RV1" V 8345 2150 50  0000 C CNN
 F 1 "50K" V 8436 2150 50  0000 C CNN
-F 2 "OpenOpParts:RV100F-30-4K1-B50K" H 8550 2150 50  0001 C CNN
+F 2 "teensy_beats_parts:RV100F-30-4K1-B50K" H 8550 2150 50  0001 C CNN
 F 3 "~" H 8550 2150 50  0001 C CNN
 	1    8550 2150
@@
 F 0 "MK1" H 7130 4646 50  0000 L CNN
 F 1 "Microphone_Condenser" H 7130 4555 50  0000 L CNN
-F 2 "OpenOpParts:AOM-6738P-R" V 7000 4700 50  0001 C CNN
+F 2 "teensy_beats_parts:AOM-6738P-R" V 7000 4700 50  0001 C CNN
 F 3 "~" V 7000 4700 50  0001 C CNN
 	1    7000 4600
