File: boost_and_charge.sch (KiCad schematic (older format))
At the start: 36 parts, among them J1 Conn_01x02_Female, SW5 SW_Push, U4 MCP73871, U5 TPS61090

Commit message: mass rename
Parts:
- TP1, TP2, TP3, TP4, TP5: footprint OpenOpParts:TestPoint1mm -> teensy_beats_parts:TestPoint1mm
Changed lines of the file:
@@
 F 0 "TP1" V 5095 6174 50  0000 C CNN
 F 1 "TestPoint" V 5004 6174 50  0000 C CNN
-F 2 "OpenOpParts:TestPoint1mm" H 5100 6100 50  0001 C CNN
+F 2 "teensy_beats_parts:TestPoint1mm" H 5100 6100 50  0001 C CNN
 F 3 "~" H 5100 6100 50  0001 C CNN
 	1    4900 6100
@@
 F 0 "TP2" V 5095 6374 50  0000 C CNN
 F 1 "TestPoint" V 5004 6374 50  0000 C CNN
-F 2 "OpenOpParts:TestPoint1mm" H 5100 6300 50  0001 C CNN
+F 2 "teensy_beats_parts:TestPoint1mm" H 5100 6300 50  0001 C CNN
 F 3 "~" H 5100 6300 50  0001 C CNN
 	1    4900 6300
@@
 F 0 "TP3" V 5095 6624 50  0000 C CNN
 F 1 "TestPoint" V 5004 6624 50  0000 C CNN
-F 2 "OpenOpParts:TestPoint1mm" H 5100 6550 50  0001 C CNN
+F 2 "teensy_beats_parts:TestPoint1mm" H 5100 6550 50  0001 C CNN
 F 3 "~" H 5100 6550 50  0001 C CNN
 	1    4900 6550
@@
 F 0 "TP5" V 5095 7024 50  0000 C CNN
 F 1 "TestPoint" V 5004 7024 50  0000 C CNN
-F 2 "OpenOpParts:TestPoint1mm" H 5100 6950 50  0001 C CNN
+F 2 "teensy_beats_parts:TestPoint1mm" H 5100 6950 50  0001 C CNN
 F 3 "~" H 5100 6950 50  0001 C CNN
 	1    4900 6950
@@
 F 0 "TP4" V 5095 6824 50  0000 C CNN
 F 1 "TestPoint" V 5004 6824 50  0000 C CNN
-F 2 "OpenOpParts:TestPoint1mm" H 5100 6750 50  0001 C CNN
+F 2 "teensy_beats_parts:TestPoint1mm" H 5100 6750 50  0001 C CNN
 F 3 "~" H 5100 6750 50  0001 C CNN
 	1    4900 6750
