File: keypad.sch (KiCad schematic (older format))
At the start: 80 parts, among them Q1 BSS138, Q2 BSS138, SW1 Rotary_Encoder_Switch, SW2 Rotary_Encoder_Switch, SW3 Rotary_Encoder_Switch, SW4 Rotary_Encoder_Switch

Commit message: mass rename
Parts:
- LED1, LED10, LED11, LED12, LED13, LED14, LED15, LED16, LED17, LED18, LED19, LED2, LED20, LED3, LED4, LED5, LED6, LED7, LED8, LED9: footprint OpenOpParts:APA102C-2020 -> teensy_beats_parts:APA102C-2020; symbol OpenOpParts:APA102C -> teensy_beats_parts:APA102C
- SW1, SW2, SW3, SW4: footprint OpenOpParts:Bourns-SMD-Encoder -> teensy_beats_parts:Bourns-SMD-Encoder
Changed lines of the file:
@@
 F 0 "SW4" V 3900 2320 50  0000 R CNN
 F 1 "Rotary_Encoder_Switch" V 3945 2320 50  0001 R CNN
-F 2 "OpenOpParts:Bourns-SMD-Encoder" H 3750 2710 50  0001 C CNN
+F 2 "teensy_beats_parts:Bourns-SMD-Encoder" H 3750 2710 50  0001 C CNN
 F 3 "~" H 3900 2810 50  0001 C CNN
 	1    3900 2550
@@
 F 0 "SW3" V 3200 2320 50  0000 R CNN
 F 1 "Rotary_Encoder_Switch" V 3245 2320 50  0001 R CNN
-F 2 "OpenOpParts:Bourns-SMD-Encoder" H 3050 2710 50  0001 C CNN
+F 2 "teensy_beats_parts:Bourns-SMD-Encoder" H 3050 2710 50  0001 C CNN
 F 3 "~" H 3200 2810 50  0001 C CNN
 	1    3200 2550
@@
 F 0 "SW2" V 2500 2250 50  0000 C CNN
 F 1 "Rotary_Encoder_Switch" V 2400 3900 50  0001 C CNN
-F 2 "OpenOpParts:Bourns-SMD-Encoder" H 2350 2710 50  0001 C CNN
+F 2 "teensy_beats_parts:Bourns-SMD-Encoder" H 2350 2710 50  0001 C CNN
 F 3 "~" H 2500 2810 50  0001 C CNN
 	1    2500 2550
@@
 F 0 "SW1" V 1800 2320 50  0000 R CNN
 F 1 "Rotary_Encoder_Switch" V 1845 2320 50  0001 R CNN
-F 2 "OpenOpParts:Bourns-SMD-Encoder" H 1650 2710 50  0001 C CNN
+F 2 "teensy_beats_parts:Bourns-SMD-Encoder" H 1650 2710 50  0001 C CNN
 F 3 "~" H 1800 2810 50  0001 C CNN
 	1    1800 2550
@@
 	3700 4550 3700 4650
 $Comp
-L OpenOpParts:APA102C LED5
+L teensy_beats_parts:APA102C LED5
 U 1 1 5BB9BD6C
 P 10300 2600
 F 0 "LED5" H 10300 2965 50  0000 C CNN
 F 1 "APA102C" H 10300 2874 50  0000 C CNN
-F 2 "OpenOpParts:APA102C-2020" H 10300 2600 50  0001 C CNN
+F 2 "teensy_beats_parts:APA102C-2020" H 10300 2600 50  0001 C CNN
 F 3 "" H 10300 2600 50  0001 C CNN
 	1    10300 2600
@@
 $EndComp
 $Comp
-L OpenOpParts:APA102C LED4
+L teensy_beats_parts:APA102C LED4
 U 1 1 5BB9BE03
 P 9200 2600
 F 0 "LED4" H 9200 2965 50  0000 C CNN
 F 1 "APA102C" H 9200 2874 50  0000 C CNN
-F 2 "OpenOpParts:APA102C-2020" H 9200 2600 50  0001 C CNN
+F 2 "teensy_beats_parts:APA102C-2020" H 9200 2600 50  0001 C CNN
 F 3 "" H 9200 2600 50  0001 C CNN
 	1    9200 2600
@@
 $EndComp
 $Comp
-L OpenOpParts:APA102C LED3
+L teensy_beats_parts:APA102C LED3
 U 1 1 5BB9BE98
 P 8100 2600
 F 0 "LED3" H 8100 2965 50  0000 C CNN
 F 1 "APA102C" H 8100 2874 50  0000 C CNN
-F 2 "OpenOpParts:APA102C-2020" H 8100 2600 50  0001 C CNN
+F 2 "teensy_beats_parts:APA102C-2020" H 8100 2600 50  0001 C CNN
 F 3 "" H 8100 2600 50  0001 C CNN
 	1    8100 2600
@@
 $EndComp
 $Comp
-L OpenOpParts:APA102C LED2
+L teensy_beats_parts:APA102C LED2
 U 1 1 5BB9BF41
 P 7000 2600
 F 0 "LED2" H 7000 2965 50  0000 C CNN
 F 1 "APA102C" H 7000 2874 50  0000 C CNN
-F 2 "OpenOpParts:APA102C-2020" H 7000 2600 50  0001 C CNN
+F 2 "teensy_beats_parts:APA102C-2020" H 7000 2600 50  0001 C CNN
 F 3 "" H 7000 2600 50  0001 C CNN
 	1    7000 2600
@@
 $EndComp
 $Comp
-L OpenOpParts:APA102C LED1
+L teensy_beats_parts:APA102C LED1
 U 1 1 5BB9D835
 P 5900 2600
 F 0 "LED1" H 5900 2965 50  0000 C CNN
 F 1 "APA102C" H 5900 2874 50  0000 C CNN
-F 2 "OpenOpParts:APA102C-2020" H 5900 2600 50  0001 C CNN
+F 2 "teensy_beats_parts:APA102C-2020" H 5900 2600 50  0001 C CNN
 F 3 "" H 5900 2600 50  0001 C CNN
 	1    5900 2600
@@
 $EndComp
 $Comp
-L OpenOpParts:APA102C LED10
+L teensy_beats_parts:APA102C LED10
 U 1 1 5BBBF02B
 P 10300 3500
 F 0 "LED10" H 10300 3865 50  0000 C CNN
 F 1 "APA102C" H 10300 3774 50  0000 C CNN
-F 2 "OpenOpParts:APA102C-2020" H 10300 3500 50  0001 C CNN
+F 2 "teensy_beats_parts:APA102C-2020" H 10300 3500 50  0001 C CNN
 F 3 "" H 10300 3500 50  0001 C CNN
 	1    10300 3500
@@
 $EndComp
 $Comp
-L OpenOpParts:APA102C LED9
+L teensy_beats_parts:APA102C LED9
 U 1 1 5BBBF032
 P 9200 3500
 F 0 "LED9" H 9200 3865 50  0000 C CNN
 F 1 "APA102C" H 9200 3774 50  0000 C CNN
-F 2 "OpenOpParts:APA102C-2020" H 9200 3500 50  0001 C CNN
+F 2 "teensy_beats_parts:APA102C-2020" H 9200 3500 50  0001 C CNN
 F 3 "" H 9200 3500 50  0001 C CNN
 	1    9200 3500
@@
 $EndComp
 $Comp
-L OpenOpParts:APA102C LED8
+L teensy_beats_parts:APA102C LED8
 U 1 1 5BBBF039
 P 8100 3500
 F 0 "LED8" H 8100 3865 50  0000 C CNN
 F 1 "APA102C" H 8100 3774 50  0000 C CNN
-F 2 "OpenOpParts:APA102C-2020" H 8100 3500 50  0001 C CNN
+F 2 "teensy_beats_parts:APA102C-2020" H 8100 3500 50  0001 C CNN
 F 3 "" H 8100 3500 50  0001 C CNN
 	1    8100 3500
@@
 $EndComp
 $Comp
-L OpenOpParts:APA102C LED7
+L teensy_beats_parts:APA102C LED7
 U 1 1 5BBBF040
 P 7000 3500
 F 0 "LED7" H 7000 3865 50  0000 C CNN
 F 1 "APA102C" H 7000 3774 50  0000 C CNN
-F 2 "OpenOpParts:APA102C-2020" H 7000 3500 50  0001 C CNN
+F 2 "teensy_beats_parts:APA102C-2020" H 7000 3500 50  0001 C CNN
 F 3 "" H 7000 3500 50  0001 C CNN
 	1    7000 3500
@@
 $EndComp
 $Comp
-L OpenOpParts:APA102C LED6
+L teensy_beats_parts:APA102C LED6
 U 1 1 5BBBF047
 P 5900 3500
 F 0 "LED6" H 5900 3865 50  0000 C CNN
 F 1 "APA102C" H 5900 3774 50  0000 C CNN
-F 2 "OpenOpParts:APA102C-2020" H 5900 3500 50  0001 C CNN
+F 2 "teensy_beats_parts:APA102C-2020" H 5900 3500 50  0001 C CNN
 F 3 "" H 5900 3500 50  0001 C CNN
 	1    5900 3500
@@
 $EndComp
 $Comp
-L OpenOpParts:APA102C LED15
+L teensy_beats_parts:APA102C LED15
 U 1 1 5BBC2504
 P 10300 4400
 F 0 "LED15" H 10300 4765 50  0000 C CNN
 F 1 "APA102C" H 10300 4674 50  0000 C CNN
-F 2 "OpenOpParts:APA102C-2020" H 10300 4400 50  0001 C CNN
+F 2 "teensy_beats_parts:APA102C-2020" H 10300 4400 50  0001 C CNN
 F 3 "" H 10300 4400 50  0001 C CNN
 	1    10300 4400
@@
 $EndComp
 $Comp
-L OpenOpParts:APA102C LED14
+L teensy_beats_parts:APA102C LED14
 U 1 1 5BBC250B
 P 9200 4400
 F 0 "LED14" H 9200 4765 50  0000 C CNN
 F 1 "APA102C" H 9200 4674 50  0000 C CNN
-F 2 "OpenOpParts:APA102C-2020" H 9200 4400 50  0001 C CNN
+F 2 "teensy_beats_parts:APA102C-2020" H 9200 4400 50  0001 C CNN
 F 3 "" H 9200 4400 50  0001 C CNN
 	1    9200 4400
@@
 $EndComp
 $Comp
-L OpenOpParts:APA102C LED13
+L teensy_beats_parts:APA102C LED13
 U 1 1 5BBC2512
 P 8100 4400
 F 0 "LED13" H 8100 4765 50  0000 C CNN
 F 1 "APA102C" H 8100 4674 50  0000 C CNN
-F 2 "OpenOpParts:APA102C-2020" H 8100 4400 50  0001 C CNN
+F 2 "teensy_beats_parts:APA102C-2020" H 8100 4400 50  0001 C CNN
 F 3 "" H 8100 4400 50  0001 C CNN
 	1    8100 4400
@@
 $EndComp
 $Comp
-L OpenOpParts:APA102C LED12
+L teensy_beats_parts:APA102C LED12
 U 1 1 5BBC2519
 P 7000 4400
 F 0 "LED12" H 7000 4765 50  0000 C CNN
 F 1 "APA102C" H 7000 4674 50  0000 C CNN
-F 2 "OpenOpParts:APA102C-2020" H 7000 4400 50  0001 C CNN
+F 2 "teensy_beats_parts:APA102C-2020" H 7000 4400 50  0001 C CNN
 F 3 "" H 7000 4400 50  0001 C CNN
 	1    7000 4400
@@
 $EndComp
 $Comp
-L OpenOpParts:APA102C LED11
+L teensy_beats_parts:APA102C LED11
 U 1 1 5BBC2520
 P 5900 4400
 F 0 "LED11" H 5900 4765 50  0000 C CNN
 F 1 "APA102C" H 5900 4674 50  0000 C CNN
-F 2 "OpenOpParts:APA102C-2020" H 5900 4400 50  0001 C CNN
+F 2 "teensy_beats_parts:APA102C-2020" H 5900 4400 50  0001 C CNN
 F 3 "" H 5900 4400 50  0001 C CNN
 	1    5900 4400
@@
 $EndComp
 $Comp
-L OpenOpParts:APA102C LED20
+L teensy_beats_parts:APA102C LED20
 U 1 1 5BBC75A4
 P 10300 5300
 F 0 "LED20" H 10300 5665 50  0000 C CNN
 F 1 "APA102C" H 10300 5574 50  0000 C CNN
-F 2 "OpenOpParts:APA102C-2020" H 10300 5300 50  0001 C CNN
+F 2 "teensy_beats_parts:APA102C-2020" H 10300 5300 50  0001 C CNN
 F 3 "" H 10300 5300 50  0001 C CNN
 	1    10300 5300
@@
 $EndComp
 $Comp
-L OpenOpParts:APA102C LED19
+L teensy_beats_parts:APA102C LED19
 U 1 1 5BBC75AB
 P 9200 5300
 F 0 "LED19" H 9200 5665 50  0000 C CNN
 F 1 "APA102C" H 9200 5574 50  0000 C CNN
-F 2 "OpenOpParts:APA102C-2020" H 9200 5300 50  0001 C CNN
+F 2 "teensy_beats_parts:APA102C-2020" H 9200 5300 50  0001 C CNN
 F 3 "" H 9200 5300 50  0001 C CNN
 	1    9200 5300
@@
 $EndComp
 $Comp
-L OpenOpParts:APA102C LED18
+L teensy_beats_parts:APA102C LED18
 U 1 1 5BBC75B2
 P 8100 5300
 F 0 "LED18" H 8100 5665 50  0000 C CNN
 F 1 "APA102C" H 8100 5574 50  0000 C CNN
-F 2 "OpenOpParts:APA102C-2020" H 8100 5300 50  0001 C CNN
+F 2 "teensy_beats_parts:APA102C-2020" H 8100 5300 50  0001 C CNN
 F 3 "" H 8100 5300 50  0001 C CNN
 	1    8100 5300
@@
 $EndComp
 $Comp
-L OpenOpParts:APA102C LED17
+L teensy_beats_parts:APA102C LED17
 U 1 1 5BBC75B9
 P 7000 5300
 F 0 "LED17" H 7000 5665 50  0000 C CNN
 F 1 "APA102C" H 7000 5574 50  0000 C CNN
-F 2 "OpenOpParts:APA102C-2020" H 7000 5300 50  0001 C CNN
+F 2 "teensy_beats_parts:APA102C-2020" H 7000 5300 50  0001 C CNN
 F 3 "" H 7000 5300 50  0001 C CNN
 	1    7000 5300
@@
 $EndComp
 $Comp
-L OpenOpParts:APA102C LED16
+L teensy_beats_parts:APA102C LED16
 U 1 1 5BBC75C0
 P 5900 5300
 F 0 "LED16" H 5900 5665 50  0000 C CNN
 F 1 "APA102C" H 5900 5574 50  0000 C CNN
-F 2 "OpenOpParts:APA102C-2020" H 5900 5300 50  0001 C CNN
+F 2 "teensy_beats_parts:APA102C-2020" H 5900 5300 50  0001 C CNN
 F 3 "" H 5900 5300 50  0001 C CNN
 	1    5900 5300
