File: teensy_beats.kicad_pcb (KiCad board)
At the start: 2 copper layers, 86.4 x 110 mm, 143 parts, among them J1 Conn_01x02_Female, J2 AudioJack3_Ground, J3 Conn_01x04_Male, Q1 BSS138, Q2 BSS138, SW1 Rotary_Encoder_Switch, SW2 Rotary_Encoder_Switch, SW3 Rotary_Encoder_Switch, SW4 Rotary_Encoder_Switch, SW5 SW_Push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

Commit message: mass rename
Parts:
- J2: footprint OpenOpParts:SJ1-3523N -> teensy_beats_parts:SJ1-3523N
- LED1, LED10, LED11, LED12, LED13, LED14, LED15, LED16, LED17, LED18, LED19, LED2, LED20, LED3, LED4, LED5, LED6, LED7, LED8, LED9: footprint OpenOpParts:APA102C-2020 -> teensy_beats_parts:APA102C-2020
- MK1: footprint OpenOpParts:AOM-6738P-R -> teensy_beats_parts:AOM-6738P-R
- RV1: footprint OpenOpParts:RV100F-30-4K1-B50K -> teensy_beats_parts:RV100F-30-4K1-B50K
- SW1, SW2, SW3, SW4: footprint OpenOpParts:Bourns-SMD-Encoder -> teensy_beats_parts:Bourns-SMD-Encoder
- TP1, TP2, TP3, TP4, TP5: footprint OpenOpParts:TestPoint1mm -> teensy_beats_parts:TestPoint1mm
- U1: footprint OpenOpParts:Teensy35_36 -> teensy_beats_parts:Teensy35_36
- U3: footprint OpenOpParts:2.4inTFT_TOUCH_SPI -> teensy_beats_parts:2.4inTFT_TOUCH_SPI
Changed lines of the file:
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@@
     (add_net VPCC)
   )
-  (module OpenOpParts:2.4inTFT_TOUCH_SPI (layer F.Cu)
+  (module teensy_beats_parts:2.4inTFT_TOUCH_SPI (layer F.Cu)
     (at 95.4 58.64)
     (fp_text reference U3 (at -32.26 -13.87) (layer F.SilkS)
@@
       (net 54 TOUCH_IRQ))
   )
-  (module OpenOpParts:Teensy35_36 (layer F.Cu)
+  (module teensy_beats_parts:Teensy35_36 (layer F.Cu)
     (at 112 58.75 180)
     (fp_text reference U1 (at 0.95 0.075 180) (layer F.SilkS)
@@
       (net 9 +3V3))
   )
-  (module OpenOpParts:TestPoint1mm (layer B.Cu)
+  (module teensy_beats_parts:TestPoint1mm (layer B.Cu)
     (at 134.025 86.075)
     (zone_connect 2)
@@
       (net 7 GND) (zone_connect 2))
   )
-  (module OpenOpParts:TestPoint1mm (layer B.Cu)
+  (module teensy_beats_parts:TestPoint1mm (layer B.Cu)
     (at 104.875 48.95)
     (zone_connect 2)
@@
       (net 9 +3V3) (zone_connect 2))
   )
-  (module OpenOpParts:TestPoint1mm (layer B.Cu)
+  (module teensy_beats_parts:TestPoint1mm (layer B.Cu)
     (at 132.25 84.075)
     (zone_connect 2)
@@
       (net 8 +5V) (zone_connect 2))
   )
-  (module OpenOpParts:TestPoint1mm (layer F.Cu)
+  (module teensy_beats_parts:TestPoint1mm (layer F.Cu)
     (at 118.875 71.775)
     (zone_connect 2)
@@
       (net 133 PG) (zone_connect 2))
   )
-  (module OpenOpParts:TestPoint1mm (layer F.Cu)
+  (module teensy_beats_parts:TestPoint1mm (layer F.Cu)
     (at 130.6 70.425)
     (zone_connect 2)
@@
     )
   )
-  (module OpenOpParts:SJ1-3523N (layer F.Cu)
+  (module teensy_beats_parts:SJ1-3523N (layer F.Cu)
     (at 90 37.29 270)
     (fp_text reference J2 (at 6.635 2.675) (layer F.SilkS)
@@
     )
   )
-  (module OpenOpParts:Bourns-SMD-Encoder (layer F.Cu)
+  (module teensy_beats_parts:Bourns-SMD-Encoder (layer F.Cu)
     (at 73 91 180)
     (fp_text reference SW1 (at -8.4 -3.475 180) (layer F.SilkS)
@@
     (pad "" np_thru_hole circle (at 0 0 180) (size 2.05 2.05) (drill 2.05) (layers *.Cu *.Mask))
   )
-  (module OpenOpParts:Bourns-SMD-Encoder (layer F.Cu)
+  (module teensy_beats_parts:Bourns-SMD-Encoder (layer F.Cu)
     (at 109 91 180)
     (fp_text reference SW3 (at -8.475 -3.4 180) (layer F.SilkS)
@@
     (pad "" np_thru_hole circle (at 0 0 180) (size 2.05 2.05) (drill 2.05) (layers *.Cu *.Mask))
   )
-  (module OpenOpParts:Bourns-SMD-Encoder (layer F.Cu)
+  (module teensy_beats_parts:Bourns-SMD-Encoder (layer F.Cu)
     (at 91 91 180)
     (fp_text reference SW2 (at -8.4 -3.4 180) (layer F.SilkS)
@@
     (pad "" np_thru_hole circle (at 0 0 180) (size 2.05 2.05) (drill 2.05) (layers *.Cu *.Mask))
   )
-  (module OpenOpParts:Bourns-SMD-Encoder (layer F.Cu)
+  (module teensy_beats_parts:Bourns-SMD-Encoder (layer F.Cu)
     (at 127 91 180)
     (fp_text reference SW4 (at -8.375 -3.5 180) (layer F.SilkS)
@@
     )
   )
-  (module OpenOpParts:AOM-6738P-R (layer F.Cu)
+  (module teensy_beats_parts:AOM-6738P-R (layer F.Cu)
     (at 138.1 44.75 90)
     (fp_text reference MK1 (at 0.075 0.2 90) (layer F.SilkS)
@@
     )
   )
-  (module OpenOpParts:APA102C-2020 (layer F.Cu)
+  (module teensy_beats_parts:APA102C-2020 (layer F.Cu)
     (at 88 114)
     (solder_mask_margin 0.05)
@@
       (net 109 "Net-(LED7-Pad5)"))
   )
-  (module OpenOpParts:APA102C-2020 (layer F.Cu)
+  (module teensy_beats_parts:APA102C-2020 (layer F.Cu)
     (at 124 103 180)
     (solder_mask_margin 0.05)
@@
       (net 46 "Net-(LED1-Pad5)"))
   )
-  (module OpenOpParts:APA102C-2020 (layer F.Cu)
+  (module teensy_beats_parts:APA102C-2020 (layer F.Cu)
     (at 112 103 180)
     (solder_mask_margin 0.05)
@@
       (net 101 "Net-(LED2-Pad5)"))
   )
-  (module OpenOpParts:APA102C-2020 (layer F.Cu)
+  (module teensy_beats_parts:APA102C-2020 (layer F.Cu)
     (at 124 136)
     (solder_mask_margin 0.05)
@@
       (net 42 "Net-(LED11-Pad2)"))
   )
-  (module OpenOpParts:APA102C-2020 (layer F.Cu)
+  (module teensy_beats_parts:APA102C-2020 (layer F.Cu)
     (at 112 136)
     (solder_mask_margin 0.05)
@@
       (net 91 "Net-(LED19-Pad5)"))
   )
-  (module OpenOpParts:APA102C-2020 (layer F.Cu)
+  (module teensy_beats_parts:APA102C-2020 (layer F.Cu)
     (at 100 136)
     (solder_mask_margin 0.05)
@@
       (net 93 "Net-(LED18-Pad5)"))
   )
-  (module OpenOpParts:APA102C-2020 (layer F.Cu)
+  (module teensy_beats_parts:APA102C-2020 (layer F.Cu)
     (at 88 136)
     (solder_mask_margin 0.05)
@@
       (net 95 "Net-(LED17-Pad5)"))
   )
-  (module OpenOpParts:APA102C-2020 (layer F.Cu)
+  (module teensy_beats_parts:APA102C-2020 (layer F.Cu)
     (at 76 136)
     (solder_mask_margin 0.05)
@@
       (net 89 "Net-(LED16-Pad5)"))
   )
-  (module OpenOpParts:APA102C-2020 (layer F.Cu)
+  (module teensy_beats_parts:APA102C-2020 (layer F.Cu)
     (at 76 125 180)
     (solder_mask_margin 0.05)
@@
       (net 99 "Net-(LED15-Pad5)"))
   )
-  (module OpenOpParts:APA102C-2020 (layer F.Cu)
+  (module teensy_beats_parts:APA102C-2020 (layer F.Cu)
     (at 88 125 180)
     (solder_mask_margin 0.05)
@@
       (net 98 "Net-(LED14-Pad5)"))
   )
-  (module OpenOpParts:APA102C-2020 (layer F.Cu)
+  (module teensy_beats_parts:APA102C-2020 (layer F.Cu)
     (at 100 125 180)
     (solder_mask_margin 0.05)
@@
       (net 117 "Net-(LED13-Pad5)"))
   )
-  (module OpenOpParts:APA102C-2020 (layer F.Cu)
+  (module teensy_beats_parts:APA102C-2020 (layer F.Cu)
     (at 112 125 180)
     (solder_mask_margin 0.05)
@@
       (net 115 "Net-(LED12-Pad5)"))
   )
-  (module OpenOpParts:APA102C-2020 (layer F.Cu)
+  (module teensy_beats_parts:APA102C-2020 (layer F.Cu)
     (at 124 125 180)
     (solder_mask_margin 0.05)
@@
       (net 113 "Net-(LED11-Pad5)"))
   )
-  (module OpenOpParts:APA102C-2020 (layer F.Cu)
+  (module teensy_beats_parts:APA102C-2020 (layer F.Cu)
     (at 124 114)
     (solder_mask_margin 0.05)
@@
       (net 39 "Net-(LED1-Pad2)"))
   )
-  (module OpenOpParts:APA102C-2020 (layer F.Cu)
+  (module teensy_beats_parts:APA102C-2020 (layer F.Cu)
     (at 112 114)
     (solder_mask_margin 0.05)
@@
       (net 38 "Net-(LED10-Pad2)"))
   )
-  (module OpenOpParts:APA102C-2020 (layer F.Cu)
+  (module teensy_beats_parts:APA102C-2020 (layer F.Cu)
     (at 100 114)
     (solder_mask_margin 0.05)
@@
       (net 111 "Net-(LED8-Pad5)"))
   )
-  (module OpenOpParts:APA102C-2020 (layer F.Cu)
+  (module teensy_beats_parts:APA102C-2020 (layer F.Cu)
     (at 76 114)
     (solder_mask_margin 0.05)
@@
       (net 107 "Net-(LED6-Pad5)"))
   )
-  (module OpenOpParts:APA102C-2020 (layer F.Cu)
+  (module teensy_beats_parts:APA102C-2020 (layer F.Cu)
     (at 76 103 180)
     (solder_mask_margin 0.05)
@@
       (net 131 RGB_CLOCK_HIGH))
   )
-  (module OpenOpParts:APA102C-2020 (layer F.Cu)
+  (module teensy_beats_parts:APA102C-2020 (layer F.Cu)
     (at 88 103 180)
     (solder_mask_margin 0.05)
@@
       (net 105 "Net-(LED4-Pad5)"))
   )
-  (module OpenOpParts:APA102C-2020 (layer F.Cu)
+  (module teensy_beats_parts:APA102C-2020 (layer F.Cu)
     (at 100 103 180)
     (solder_mask_margin 0.05)
@@
     )
   )
-  (module OpenOpParts:RV100F-30-4K1-B50K (layer F.Cu)
+  (module teensy_beats_parts:RV100F-30-4K1-B50K (layer F.Cu)
     (at 75 42.25)
     (fp_text reference RV1 (at 0.06 4.8) (layer F.SilkS)
