File: teensy_beats.sch (KiCad schematic (older format))
At the start: 6 parts, among them J3 Conn_01x04_Male, U1 Teensy3.6, U2 M25PX32-VMW, U3 TFT_TOUCH_SPI

Commit message: mass rename
Parts:
- U1: footprint OpenOpParts:Teensy35_36 -> teensy_beats_parts:Teensy35_36; symbol OpenOpParts:TEENSY3.6-OpenOp -> teensy_beats_parts:TEENSY3.6-teensy_beats
- U3: footprint OpenOpParts:2.4inTFT_TOUCH_SPI -> teensy_beats_parts:2.4inTFT_TOUCH_SPI; symbol OpenOpParts:TFT_TOUCH_SPI -> teensy_beats_parts:TFT_TOUCH_SPI
Changed lines of the file:
@@
 EESchema Schematic File Version 4
-LIBS:Open Op-cache
+LIBS:teensy_beats-cache
 EELAYER 26 0
 EELAYER END
@@
 	6350 4700 7150 4700
 $Comp
-L OpenOpParts:TFT_TOUCH_SPI U3
+L teensy_beats_parts:TFT_TOUCH_SPI U3
 U 1 1 5BA764CE
 P 9600 4800
 F 0 "U3" H 9681 5715 50  0000 C CNN
 F 1 "TFT_TOUCH_SPI" H 9681 5624 50  0000 C CNN
-F 2 "OpenOpParts:2.4inTFT_TOUCH_SPI" H 9600 3950 50  0001 C CNN
+F 2 "teensy_beats_parts:2.4inTFT_TOUCH_SPI" H 9600 3950 50  0001 C CNN
 F 3 "" H 9600 3950 50  0001 C CNN
 	1    9600 4800
@@
 VOLUME
 $Comp
-L OpenOpParts:TEENSY3.6-OpenOp U1
+L teensy_beats_parts:TEENSY3.6-teensy_beats U1
 U 1 1 5B903484
 P 4300 2850
 F 0 "U1" H 4300 5237 60  0000 C CNN
 F 1 "Teensy3.6" H 4300 5131 60  0000 C CNN
-F 2 "OpenOpParts:Teensy35_36" H 4300 2850 60  0001 C CNN
+F 2 "teensy_beats_parts:Teensy35_36" H 4300 2850 60  0001 C CNN
 F 3 "" H 4300 2850 60  0000 C CNN
 	1    4300 2850
