File: hardware/teensy_beats.sch (KiCad schematic (older format))
At the start: 6 parts, among them J3 Conn_01x04_Male, U1 Teensy3.6, U2 M25PX32-VMW, U3 TFT_TOUCH_SPI

Commit message: changed pin mapping to add pg signal, added enable jumper for development. adding updated gerbers.
Connections:
- net labels added: PG
Changed lines of the file:
@@
 Text GLabel 5300 4550 2    50   Input ~ 0
 TFT_CS
-Text GLabel 5300 4650 2    50   Input ~ 0
+Text GLabel 3300 1850 0    50   Input ~ 0
 TFT_DC
 Text GLabel 3300 2650 0    50   Input ~ 0
@@
 Text GLabel 5300 4950 2    50   Input ~ 0
 E2A
-Text GLabel 3300 1850 0    50   Input ~ 0
+Text GLabel 3300 1650 0    50   Input ~ 0
 E3B
 Text GLabel 3300 2250 0    50   Input ~ 0
@@
 	1    0    0    -1
 $EndComp
+Text GLabel 5300 4650 2    50   Input ~ 0
+PG
 $EndSCHEMATC
