File: hardware/teensy_beats.sch (KiCad schematic (older format))
At the start: 12 parts, among them J3 Conn_01x04_Male, J5 USB_B_Micro, J6 USB_A, J7 Micro_SD_Card, U2 M25PX32-VMW, U3 TFT_TOUCH_SPI, U8 MK66FX1M0VMD18, U9 MKL02Z32VFG4

Commit message: v2 mostly routed
Parts:
- removed J3: Conn_01x04_Male, Connectors_JST:JST_SH_BM04B-SRSS-TB_04x1.00mm_Straight, symbol Connector:Conn_01x04_Male
- removed J5: USB_B_Micro, Connector_USB:USB_Micro-B_Wuerth_629105150521, symbol Connector:USB_B_Micro
- removed J6: USB_A, digikey-footprints:USB_A_Female_AU-Y1006-3, symbol Connector:USB_A
- removed J7: Micro_SD_Card, Connector_Card:microSD_HC_Wuerth_693072010801, symbol Connector:Micro_SD_Card
- removed R31, R32: 33, Resistor_SMD:R_0805_2012Metric, symbol Device:R_Small
- removed U8: MK66FX1M0VMD18, teensy_beats_parts:BGA144C100P12X12_1300X1300X170, symbol MK66FX1M0VMD18:MK66FX1M0VMD18
- removed U9: MKL02Z32VFG4, teensy_beats_parts:QFN50P300X300X65-17N, symbol MKL02Z32VFG4:MKL02Z32VFG4
- added C65: 10uF, Capacitor_SMD:C_0603_1608Metric, symbol Device:C_Small
- added C66: 0.22uF, Capacitor_SMD:C_0402_1005Metric, symbol Device:C_Small
- added LS1: CMS-160916-30-3, teensy_beats_parts:SPKR_CMS-160916-30-3, symbol CMS-160916-30-3:CMS-160916-30-3
- added R35: 1M, Resistor_SMD:R_0402_1005Metric, symbol Device:R
- added U11: MAX98357AETE+T, teensy_beats_parts:QFN50P300X300X80-17N, symbol MAX98357AETE_T:MAX98357AETE+T
- R1, R2: footprint Resistors_SMD:R_0805 -> Resistor_SMD:R_0402_1005Metric
Connections:
- net labels added: BCLK2, DIN, DOUT, DOUT2, LRCLK2, PHONE_DET
- net labels removed: RESET, RX, TX, VBUS
- wire segments 68 -> 84
Other:
- note added: "Backlight PWM?"
