File: hardware/SGTL5000.sch (KiCad schematic (older format))
At the start: 20 parts, among them J2 AudioJack3_Ground, U6 AP7313-1.8V, U7 SGTL5000

Commit message: v2 mostly routed
Parts:
- removed J2: AudioJack3_Ground, teensy_beats_parts:SJ1-3523N, symbol teensy_beats_parts:SJ1-3523N
- added J2: Switched, teensy_beats_parts:SJ1-3525N, symbol Connector:AudioJack3_Ground_SwitchTR
- added R38: 1K, Resistor_SMD:R_0402_1005Metric, symbol Device:R
- added R39: 100K, Resistor_SMD:R_0402_1005Metric, symbol Device:R
- C26, C29, C31, C34: footprint Capacitors_SMD:C_0805 -> Capacitor_SMD:C_0805_2012Metric
- C27, C28, C30, C32, C33: footprint Capacitors_SMD:C_0805 -> Capacitor_SMD:C_0402_1005Metric
- MK1: value Microphone_Condenser -> POM-3542P-R
- R22, R23, R24, R25: footprint Resistors_SMD:R_0805 -> Resistor_SMD:R_0402_1005Metric
Connections:
- net +3V3: now also R38.1
- net at U7.2 (HPR): now also J2.R
- net at U7.4 (HPVGND): now also J2.S, R39.1
- net at U7.6 (HPL): now also J2.T, R38.2
- net RX renamed DIN
- net TX renamed DOUT
- new net PHONE_DET: J2.TN, R39.2
Other:
- moved on the sheet: C31, C32, RV1, U6
