File: hardware/keypad.sch (KiCad schematic (older format))
At the start: 80 parts, among them Q1 BSS138, Q2 BSS138, SW1 Rotary_Encoder_Switch, SW2 Rotary_Encoder_Switch, SW3 Rotary_Encoder_Switch, SW4 Rotary_Encoder_Switch

Commit message: v2 mostly routed
Parts:
- removed D1, D2, D3, D4, D5: D, Diodes_SMD:D_0805, symbol Device:D
- removed Q1, Q2: BSS138, digikey-footprints:SOT-23-3, symbol Transistor_FET:BSS138
- added D1, D2: BAS40TW, Package_TO_SOT_SMD:SOT-363_SC-70-6, symbol teensy_beats-rescue:BAS40TW-teensy_beats_parts
- added Q1: BSS138DW, Package_TO_SOT_SMD:SOT-363_SC-70-6, symbol teensy_beats-rescue:BSS138DW-teensy_beats_parts
- C1, C10, C11, C12, C13, C14, C15, C16, C17, C18, C19, C2, C20, C3, C4, C5, C6, C7, C8, C9: footprint Capacitors_SMD:C_0603 -> Capacitor_SMD:C_0402_1005Metric
- R26, R27, R28, R29: footprint Resistors_SMD:R_0805 -> Resistor_SMD:R_0402_1005Metric
- R3, R4, R5, R6, R7: value 100 -> 1000; footprint Resistors_SMD:R_0805 -> Resistor_SMD:R_0402_1005Metric
Connections:
- net +3V3: now also Q1.2 (G1), Q1.5 (G2)
- net KEYPAD_C0: now also D1.6 (A)
- net KEYPAD_C1: now also D1.5 (A)
- net KEYPAD_C2: now also D1.4 (A)
- net KEYPAD_C3: now also D2.6 (A)
- net KEYPAD_C4: now also D2.5 (A)
- net RGB_CLOCK: now also Q1.4 (S2)
- net RGB_CLOCK_HIGH: now also Q1.3 (D2)
- net RGB_DATA: now also Q1.1 (S1)
- net RGB_DATA_HIGH: now also Q1.6 (D1)
- net at S1.2, S11.2, S16.2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: now also D1.1 (K)
- net at S10.2, S15.2, S20.2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: now also D2.2 (K)
- net at S14.2, S19.2, S4.2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: now also D2.1 (K)
- net at S13.2, S18.2, S3.2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: now also D1.3 (K)
- net at S12.2, S17.2, S2.2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: now also D1.2 (K)
Other:
- moved on the sheet: R26, R27, R28, R29
