File: hardware/teensy_beats.kicad_pcb (KiCad board)
At the start: 2 copper layers, 86.4 x 110 mm, 144 parts, among them J1 Conn_01x02_Female, J2 AudioJack3_Ground, J3 Conn_01x04_Male, J4 Conn_01x02_Male, Q1 BSS138, Q2 BSS138, SW1 Rotary_Encoder_Switch, SW2 Rotary_Encoder_Switch, SW3 Rotary_Encoder_Switch, SW4 Rotary_Encoder_Switch, SW5 SW_Push, U1 Teensy3.6, U2 M25PX32-VMW, U3 TFT_TOUCH_SPI, U4 MCP73871, U5 TPS61090, U6 AP7313-1.8V, U7 SGTL5000

Commit message: start of k66 based v2 design
Parts:
- removed J3: Conn_01x04_Male, Connectors_JST:JST_SH_BM04B-SRSS-TB_04x1.00mm_Straight
- removed U1: Teensy3.6, teensy_beats_parts:Teensy35_36
- added J5: USB_B_Micro, Connector_USB:USB_Micro-B_Wuerth_629105150521, F.Cu at (105.3, 41.0)
- added J6: USB_A, digikey-footprints:USB_A_Female_AU-Y1006-3, F.Cu at (89.7, 49.8)
- added J7: Micro_SD_Card, Connector_Card:microSD_HC_Wuerth_693072010801, B.Cu at (119.2, 44.5)
- added R31: 33, Resistor_SMD:R_0805_2012Metric, F.Cu at (109.2, 46.9)
- added R32: 33, Resistor_SMD:R_0805_2012Metric, F.Cu at (109.2, 49.9)
- added U8: MK66FX1M0VMD18, teensy_beats_parts:BGA144C100P12X12_1300X1300X170, F.Cu at (108.5, 59.3)
- added U9: MKL02Z32VFG4, teensy_beats_parts:QFN50P300X300X65-17N, F.Cu at (98.3, 58.1)
- C1, C10, C11, C12, C13, C14, C15, C16, C17, C18, C19, C2, C20, C3, C4, C5, C6, C7, C8, C9: footprint Capacitors_SMD:C_0603 -> Resistor_SMD:R_0603_1608Metric
- C21, C23, C24, C25, C26, C27, C28, C29, C30, C31, C32, C33, C34, C35, C36: footprint Capacitors_SMD:C_0805 -> Resistor_SMD:R_0603_1608Metric
- R1, R10, R11, R12, R13, R14, R15, R16, R17, R18, R19, R2, R20, R21, R22, R23, R24, R25, R26, R27, R28, R29, R3, R30, R4, R5, R6, R7, R8, R9: footprint Resistors_SMD:R_0805 -> Resistor_SMD:R_0603_1608Metric
- SW5: footprint Buttons_Switches_THT:SW_Tactile_SKHH_Angled -> teensy_beats_parts:KSS231GLFS
- moved RV1 65.4 mm to (138.4, 58.4), turned to 270 degrees
- moved U2 46.1 mm to (52.6, 25.1)
- moved C26 33.0 mm to (72.0, 62.6)
- moved C28 33.0 mm to (76.2, 62.6)
- moved C31 33.0 mm to (81.8, 55.5)
- moved R22 33.0 mm to (84.6, 61.9)
- moved TP4 33.0 mm to (75.5, 64.0)
- moved U6 33.0 mm to (85.5, 55.4)
- moved C27 33.0 mm to (74.2, 62.6)
- moved C29 33.0 mm to (71.0, 57.2)
- moved C30 33.0 mm to (71.0, 55.3)
- moved L2 33.0 mm to (69.9, 62.6)
- moved R23 33.0 mm to (84.6, 59.8)
- moved U7 33.0 mm to (77.6, 57.8)
- moved J2 16.5 mm to (73.5, 37.7)
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Routing:
- net MOSI: track 93.7 -> 0.00 mm, vias 2 -> 0
- net +3V3: track 142.2 -> 60.8 mm, vias 4 -> 9
- net TFT_CS: track 79.9 -> 0.00 mm, vias 1 -> 0
- net MISO: track 79.6 -> 0.00 mm, vias 2 -> 0
- net AGND: track 77.2 -> 0.00 mm, vias 1 -> 0
- net SCLK: track 76.6 -> 0.00 mm, vias 2 -> 0
- net TFT_DC: track 68.3 -> 0.00 mm, vias 2 -> 0
- net CS: track 64.2 -> 6.27 mm, vias 2 -> 1
- net +BATT: track 111.2 -> 70.5 mm
- net LRCLK: track 44.0 -> 4.78 mm, vias 2 -> 1
- net Net-(D6-Pad3): track 66.3 -> 29.9 mm
- net E1A: track 53.4 -> 17.3 mm
- net E2A: track 48.9 -> 15.2 mm, vias 3 -> 1
- net GND: track 185.9 -> 153.9 mm, vias 285 -> 212
- net E1B: track 51.9 -> 20.6 mm
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- added copper zone on F.Cu, net +3V3
- added copper zone on PWR, net +3V3
Other:
- copper layers 2 -> 4
- rule pad_to_mask_clearance: 0.2 -> 0.05
- rule trace_min: 0.2 -> 0.127
- rule via_min_drill: 0.3 -> 0.2
- rule via_min_size: 0.4 -> 0.45

Commit message: v2 mostly routed
Parts:
- removed D4, D5: D, Diodes_SMD:D_0805
- removed D6: D_x2_KCom_AAK, digikey-footprints:SOT-23-3
- added BT1: Battery_Cell, Battery:BatteryHolder_Keystone_2462_2xAA, B.Cu at (88.7, -106.4)
- added C37: 0.22uF, Capacitor_SMD:C_0402_1005Metric, F.Cu at (163.1, 13.9)
- added C38: 0.22uF, Capacitor_SMD:C_0402_1005Metric, F.Cu at (163.3, 15.5)
- added C39: 2.2uF, Capacitor_SMD:C_0402_1005Metric, B.Cu at (97.9, 67.5)
- added C40: 4.7uF, Capacitor_SMD:C_0603_1608Metric, B.Cu at (94.9, 71.3)
- added C41: 0.22uF, Capacitor_SMD:C_0402_1005Metric, B.Cu at (97.9, 69.4)
- added C42: 0.22uF, Capacitor_SMD:C_0402_1005Metric, B.Cu at (99.5, 67.3)
- added C43: 10nF, Capacitor_SMD:C_0402_1005Metric, F.Cu at (90.0, 63.1)
- added C44: 10uF, Capacitor_SMD:C_0603_1608Metric, B.Cu at (102.6, 67.6)
- added C45: 4.7uF, Capacitor_SMD:C_0603_1608Metric, F.Cu at (108.3, 63.0)
- added C46: 0.22uF, Capacitor_SMD:C_0402_1005Metric, B.Cu at (98.1, 77.8)
- added C47: 10uF, Capacitor_SMD:C_0603_1608Metric, F.Cu at (105.8, 67.2)
- added C48: 4.7uF, Capacitor_SMD:C_0603_1608Metric, F.Cu at (109.7, 66.0)
- added C49: 0.22uF, Capacitor_SMD:C_0402_1005Metric, B.Cu at (96.3, 68.1)
- added C50: 10nF, Capacitor_SMD:C_0603_1608Metric, F.Cu at (108.1, 66.0)
- added C51: 10uF, Capacitor_SMD:C_0603_1608Metric, F.Cu at (105.0, 73.7)
- added C52: 0.22uF, Capacitor_SMD:C_0402_1005Metric, F.Cu at (108.9, 68.0)
- added C53: 0.22uF, Capacitor_SMD:C_0402_1005Metric, F.Cu at (84.8, 54.7)
- added C54: 12pF, Capacitor_SMD:C_0402_1005Metric, F.Cu at (91.8, 60.7)
- added C55: 12pF, Capacitor_SMD:C_0402_1005Metric, F.Cu at (89.5, 60.7)
- added C56: 20pF, Capacitor_SMD:C_0402_1005Metric, F.Cu at (96.4, 58.3)
- added C57: 20pF, Capacitor_SMD:C_0402_1005Metric, F.Cu at (94.1, 58.3)
- added C58: 4.7uF, Capacitor_SMD:C_0603_1608Metric, B.Cu at (94.9, 62.4)
- added C59: 0.22uF, Capacitor_SMD:C_0402_1005Metric, B.Cu at (96.3, 64.1)
- added C60: 4.7uF, Capacitor_SMD:C_0603_1608Metric, F.Cu at (115.0, 75.9)
- added C61: 0.22uF, Capacitor_SMD:C_0402_1005Metric, F.Cu at (104.3, 71.1)
- added C62: 0.22uF, Capacitor_SMD:C_0402_1005Metric, B.Cu at (93.3, 63.9)
- added C63: 0.22uF, Capacitor_SMD:C_0402_1005Metric, F.Cu at (106.3, 55.1)
- added C64: 0.22uF, Capacitor_SMD:C_0402_1005Metric, F.Cu at (87.4, 71.4)
- added C65: 10uF, Capacitor_SMD:C_0603_1608Metric, F.Cu at (136.7, 67.0)
- added C66: 0.22uF, Capacitor_SMD:C_0402_1005Metric, F.Cu at (136.5, 69.5)
- added C67: 100uF, Capacitor_SMD:C_0603_1608Metric, F.Cu at (94.3, 52.1)
- added D11: BAT54C, Package_TO_SOT_SMD:SOT-23, F.Cu at (80.6, 56.9)
- added D12: BAT54C, Package_TO_SOT_SMD:SOT-23, F.Cu at (80.6, 60.7)
- added L3: 120, Inductor_SMD:L_0603_1608Metric, F.Cu at (80.2, 54.0)
- added L4: 4.7uH, Inductor_SMD:L_1210_3225Metric, F.Cu at (105.6, 63.9)
- added LS1: CMS-160916-30-3, teensy_beats_parts:SPKR_CMS-160916-30-3, F.Cu at (138.3, 55.6)
- added Q3: DMG3415U, Package_TO_SOT_SMD:SOT-23, F.Cu at (64.5, 66.6)
- added R33: 100K, Resistor_SMD:R_0402_1005Metric, F.Cu at (87.3, -80.4)
- added R34: 100k, Resistor_SMD:R_0402_1005Metric, F.Cu at (89.1, 52.6)
- added R35: 1M, Resistor_SMD:R_0402_1005Metric, F.Cu at (135.3, 71.4)
- added R36: 10K, Resistor_SMD:R_0402_1005Metric, F.Cu at (91.3, -80.4)
- added R37: 2.2M, Resistor_SMD:R_0402_1005Metric, F.Cu at (88.0, 58.4)
- added R38: 1K, Resistor_SMD:R_0402_1005Metric, F.Cu at (105.1, 51.1)
- added R39: 100K, Resistor_SMD:R_0402_1005Metric, F.Cu at (109.1, 51.1)
- added U1: MIMXRT1062DVL6A-tbs, teensy_beats_parts:BGA196C80P14X14_1200X1200X161N, F.Cu at (97.1, 68.1)
- added U10: TPD3S014, Package_TO_SOT_SMD:SOT-23-6, F.Cu at (91.5, 52.0)
- added U11: MAX98357AETE+T, teensy_beats_parts:QFN50P300X300X80-17N, F.Cu at (133.8, 68.6)
- added Y1: 24Mhz, Oscillator:Oscillator_SMD_Abracon_ASE-4Pin_3.2x2.5mm, F.Cu at (90.7, 58.4)
- added Y2: 32.768 kHz, Crystal:Crystal_SMD_MicroCrystal_CC7V-T1A-2Pin_3.2x1.5mm, F.Cu at (95.2, 60.2)
- C1, C10, C11, C12, C13, C14, C15, C16, C17, C18, C19, C2, C20, C24, C27, C28, C3, C30, C32, C33, C4, C5, C6, C7, C8, C9: footprint Resistor_SMD:R_0603_1608Metric -> Capacitor_SMD:C_0402_1005Metric
- C21, C23, C25, C26, C29, C31, C34, C35, C36: footprint Resistor_SMD:R_0603_1608Metric -> Capacitor_SMD:C_0805_2012Metric
- C22: footprint Capacitors_SMD:C_1210 -> Capacitor_SMD:C_1210_3225Metric
- D1, D2, D3: value D -> BAS40TW; footprint Diodes_SMD:D_0805 -> Package_TO_SOT_SMD:SOT-363_SC-70-6
- J1: footprint Connectors_JST:JST_PH_S2B-PH-K_02x2.00mm_Angled -> Connector_JST:JST_PH_S2B-PH-SM4-TB_1x02-1MP_P2.00mm_Horizontal; moved to B.Cu
- J2: value AudioJack3_Ground -> Switched; footprint teensy_beats_parts:SJ1-3523N -> teensy_beats_parts:SJ1-3525N
- J5: value USB_B_Micro -> USB_C_Receptacle_USB2.0; footprint Connector_USB:USB_Micro-B_Wuerth_629105150521 -> teensy_beats_parts:MOLEX_105450-0101
- J6: value USB_A -> 629104190121; footprint digikey-footprints:USB_A_Female_AU-Y1006-3 -> teensy_beats_parts:629104190121
- MK1: value Microphone_Condenser -> POM-3542P-R
- Q1: value BSS138 -> BSS138DW; footprint digikey-footprints:SOT-23-3 -> Package_TO_SOT_SMD:SOT-363_SC-70-6
- Q2: value BSS138 -> DMG3415U; footprint digikey-footprints:SOT-23-3 -> Package_TO_SOT_SMD:SOT-23
- R1, R10, R11, R12, R13, R14, R15, R16, R17, R18, R19, R2, R20, R21, R22, R23, R24, R25, R26, R27, R28, R29, R30, R8, R9: footprint Resistor_SMD:R_0603_1608Metric -> Resistor_SMD:R_0402_1005Metric
- R3, R4, R5, R6, R7: value 100 -> 1000; footprint Resistor_SMD:R_0603_1608Metric -> Resistor_SMD:R_0402_1005Metric
- R31, R32: value 33 -> 5.1k; footprint Resistor_SMD:R_0805_2012Metric -> Resistor_SMD:R_0402_1005Metric
- TP1, TP2, U2: moved to B.Cu
- U8: value MK66FX1M0VMD18 -> W25Q64JVXGIM; footprint teensy_beats_parts:BGA144C100P12X12_1300X1300X170 -> Package_SO:SOIC-8_3.9x4.9mm_P1.27mm
- U9: value MKL02Z32VFG4 -> MKL02Z32VFG4-tbs
- moved TP4 87.9 mm to (144.8, 9.90)
- moved J1 85.3 mm to (50.2, 65.9), turned to 180 degrees
- moved R18 83.7 mm to (50.8, 82.3)
- moved TP2 69.4 mm to (63.1, 54.1), turned to 270 degrees
- moved R9 66.7 mm to (67.0, 52.2), turned to 270 degrees
- moved C35 66.4 mm to (65.4, 52.8), turned to 90 degrees
- moved RV1 66.2 mm to (74.3, 41.7), turned to 0 degrees
- moved R17 63.8 mm to (71.0, 52.2), turned to 270 degrees
- moved R8 62.4 mm to (68.2, 52.2), turned to 90 degrees
- moved R16 61.3 mm to (70.0, 52.2), turned to 90 degrees
- moved U4 56.3 mm to (69.1, 55.8), turned to 0 degrees
- moved R30 55.9 mm to (65.8, 57.3), turned to 270 degrees
- moved R11 55.1 mm to (72.8, 55.8)
- moved TP1 54.1 mm to (64.8, 70.1), turned to 270 degrees
- moved C36 53.8 mm to (72.8, 53.6), turned to 90 degrees
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Connections:
- net VLIPO renamed +VLIPO
- C23 pad 1: +BATT -> +VIN
- C24 pad 1: +BATT -> +VIN
- C35 pad 1: +BATT -> +VCHG
- D1 pad 2: KEYPAD_C0 -> Net-(D1-Pad2)
- D2 pad 2: KEYPAD_C1 -> Net-(D2-Pad2)
- D3 pad 2: KEYPAD_C2 -> (no net)
- J4 pad 1: Net-(D6-Pad3) -> Net-(D3-Pad1)
- J4 pad 2: +BATT -> +VIN
- J6 pad 1: +5V -> Net-(C67-Pad1)
- J7 pad 4: Net-(J7-Pad4) -> +3V3
- J7 pad 9: GND -> Net-(J7-Pad9)
- L1 pad 2: +BATT -> +VIN
- Q1 pad 1: +3V3 -> RGB_DATA
- Q1 pad 2: RGB_CLOCK -> +3V3
- Q2 pad 1: +3V3 -> +3V0
- Q2 pad 2: RGB_DATA -> +VIN
- Q2 pad 3: RGB_DATA_HIGH -> +VCHG
- R13 pad 1: +BATT -> +VIN
- R18 pad 2: Net-(D6-Pad3) -> Net-(D3-Pad1)
- R20 pad 1: Net-(D6-Pad1) -> Net-(D3-Pad6)
- R31 pad 1: USB0_D+ -> Net-(J5-PadB5)
- R31 pad 2: Net-(J5-Pad3) -> GND
- R32 pad 1: Net-(J5-Pad2) -> Net-(J5-PadA5)
- R32 pad 2: USB0_D- -> GND
- R8 pad 1: VBUS -> +VUSB
- S10 pad 2: Net-(D5-Pad1) -> Net-(D2-Pad2)
- S12 pad 2: Net-(D2-Pad1) -> Net-(D1-Pad2)
- S13 pad 2: Net-(D3-Pad1) -> Net-(D1-Pad3)
- S14 pad 2: Net-(D4-Pad1) -> Net-(D2-Pad1)
- S15 pad 2: Net-(D5-Pad1) -> Net-(D2-Pad2)
- S17 pad 2: Net-(D2-Pad1) -> Net-(D1-Pad2)
- S18 pad 2: Net-(D3-Pad1) -> Net-(D1-Pad3)
- S19 pad 2: Net-(D4-Pad1) -> Net-(D2-Pad1)
- S2 pad 2: Net-(D2-Pad1) -> Net-(D1-Pad2)
- S20 pad 2: Net-(D5-Pad1) -> Net-(D2-Pad2)
- S3 pad 2: Net-(D3-Pad1) -> Net-(D1-Pad3)
- S4 pad 2: Net-(D4-Pad1) -> Net-(D2-Pad1)
- S5 pad 2: Net-(D5-Pad1) -> Net-(D2-Pad2)
- S7 pad 2: Net-(D2-Pad1) -> Net-(D1-Pad2)
- S8 pad 2: Net-(D3-Pad1) -> Net-(D1-Pad3)
- S9 pad 2: Net-(D4-Pad1) -> Net-(D2-Pad1)
- SW2 pad S2: Net-(D2-Pad1) -> Net-(D1-Pad2)
- SW3 pad S2: Net-(D3-Pad1) -> Net-(D1-Pad3)
- SW4 pad S2: Net-(D4-Pad1) -> Net-(D2-Pad1)
- SW5 pad 1: Net-(D6-Pad1) -> Net-(D3-Pad6)
- SW5 pad 2: +BATT -> +VIN
- U4 pad 1: +BATT -> +VCHG
- U4 pad 17: VBUS -> +VUSB
- U4 pad 18: VBUS -> +VUSB
- U4 pad 19: VBUS -> +VUSB
- U4 pad 20: +BATT -> +VCHG
- U4 pad 3: VBUS -> +VUSB
- U4 pad 4: VBUS -> +VUSB
- U4 pad 9: VBUS -> +VUSB
- U5 pad 11: Net-(D6-Pad3) -> Net-(D3-Pad1)
- U5 pad 8: +BATT -> +VIN
- U7 pad 2: Net-(J2-Pad2) -> Net-(J2-PadR)
- U7 pad 25: RX -> DOUT
- U7 pad 26: TX -> DIN
- U7 pad 4: Net-(J2-Pad1) -> Net-(J2-PadS)
- U7 pad 6: Net-(J2-Pad3) -> Net-(J2-PadT)
- U9 pad 13: RESET -> Net-(U1-PadF13)
- U9 pad 4: RESET -> Net-(U1-PadF11)
- U9 pad 6: Net-(U8-PadJ6) -> Net-(U1-PadG13)
- U9 pad 7: Net-(U8-PadK7) -> Net-(U1-PadF14)
- U9 pad 8: Net-(U8-PadJ5) -> Net-(U1-PadF12)
- U9 pad 9: Net-(U8-PadK6) -> Net-(U1-PadM7)
Routing:
- net +5V: track 481.8 -> 266.9 mm, vias 8 -> 2
- net Net-(D4-Pad1): track 136.0 -> 0.00 mm, vias 6 -> 0
- net Net-(D5-Pad1): track 129.7 -> 0.00 mm, vias 5 -> 0
- net Net-(D2-Pad2): track 0.00 -> 129.1 mm, vias 0 -> 5
- net Net-(D1-Pad3): track 0.00 -> 116.7 mm, vias 0 -> 5
- net Net-(D3-Pad1): track 116.0 -> 0.00 mm, vias 5 -> 0
- net Net-(D1-Pad2): track 0.00 -> 100.4 mm, vias 0 -> 5
- net +VIN: track 0.00 -> 83.5 mm, vias 0 -> 1
- net MISO: track 0.00 -> 80.0 mm, vias 0 -> 2
- net MOSI: track 0.00 -> 76.7 mm, vias 0 -> 3
- net SCLK: track 0.00 -> 71.1 mm, vias 0 -> 3
- net +BATT: track 70.5 -> 0.00 mm, vias 1 -> 0
- net +VUSB: track 0.00 -> 66.0 mm
- net TFT_CS: track 0.00 -> 62.9 mm, vias 0 -> 2
- net PWR_BTN: track 6.15 -> 67.3 mm, vias 1 -> 3
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- added copper zone on F.Cu, net +5V
- added copper zone on F.Cu, net +VLIPO
- added copper zone on GND, net GND
- added copper zone on PWR, net Net-(C47-Pad1)
- added copper zone on F.Cu, net Net-(L1-Pad1)
- removed copper zone on F.Cu, net +3V3
- removed copper zone on F.Cu, net GND
Other:
- net class Default: clearance 0.2 -> 0.127
- net class OuterBGA added: clearance 0.09, trace_width 0.09, via_dia 0.45, via_drill 0.2
- rule trace_clearance: 0.2 -> 0.127
- rule trace_min: 0.127 -> 0.09
